Commit message: invert_laser & simple_navigation_goal

File: robotino_description/urdf/robotino_body.xacro (robot description, xacro)
@@ -50,5 +50,6 @@
     </anglebracketusb>
     <laser name="laser" parent="base_link">
-      <origin xyz="-0.022 0 0.232" rpy="0 0 0"/>
+      <!--origin xyz="-0.022 0 0.232" rpy="0 0 0"/-->
+      <origin xyz="0.1 0 0" rpy="0 0 0"/>
     </laser>
     <!--laser name="laser" parent="base_link"-->
