Commit message: alterações no navigation

File: robotino_description/urdf/robotino.urdf (robot description, URDF)
Before this commit: robot robotino, 8 links, 7 joints
Joints:
- joint laser_joint: origin xyz=-0.022 10 0.232 rpy=0 0 0 -> xyz=0.224 0 0.232 rpy=0 0 0

Commit message: grab_puck action server implemented, and robotino_safety, robotino.urdf, common_costmap_params.conf, map have been all modified

File: robotino_description/urdf/robotino.urdf (robot description, URDF)
Before this commit: robot robotino, 8 links, 7 joints
Joints:
- joint laser_joint: origin xyz=0.224 0 0.232 rpy=0 0 0 -> xyz=0.224 0 0.1 rpy=0 0 0
